File: Hardware/pcb.brd (EAGLE design)
At the start: 46 x 35 mm, 105 parts, among them IC1 BQ25180YBGR_BQ25180YBGR, IC2 DRV2605YZFR, IC3 BMA423_BMA423, IC9 RT6160AWSC_RT6160AWSC, J1 503480-2400_503480-2400, J2 TC2030-IDC_TC2030-IDC, J4 KH-TYPE-C-16P_KH-TYPE-C-16P, Q1 SI1308EDL-T1-GE3, Q2 20V/4.2A/52mΩ/1.4W, U1 NRF52840_QF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

Commit message: Fixed issues
Parts:
- renumbered U$13 to X1, U$6 to X2
Connections:
- net N$19 renamed P1.14
- net N$20 renamed P1.13
- net N$22 renamed P1.12
- net N$23 renamed P1.11
- net N$24 renamed P1.10
Other:
- board text removed: "**************************************************************************************************** **************************************************************************************************** **************************************************************************************************** ************************************************************************************************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"
- board text removed: ":::::::::::::::::::::::::::::::::::::::::::::::::::::::::::::::::::::::::::::::::::::::::::::::::::: :::::::::::::::::::::::::::::::::::::::::::::::::::::::::::::::::::::::::::::::::::::::::::::::::::: :::::::::::::::::::::::::::::::::::::::::::::::::::::::::::::::::::::::::::::::::::::::::::::::::::: ::::::::::::::::::::::::::::::::::::::::::::::::::::::::::::::::::::::::::::::::::::::::::::::::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"
