File: Hardware/schematic.sch (EAGLE design)
At the start: 105 parts, among them IC1 BQ25180YBGR_BQ25180YBGR, IC2 DRV2605YZFR, IC3 BMA423_BMA423, IC9 RT6160AWSC_RT6160AWSC, J1 503480-2400_503480-2400, J2 TC2030-IDC_TC2030-IDC, J4 KH-TYPE-C-16P_KH-TYPE-C-16P, Q1 SI1308EDL-T1-GE3, Q2 20V/4.2A/52mΩ/1.4W, U1 NRF52840_QF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

Commit message: Fixed issues
Parts:
- renumbered U$13 to X1, U$6 to X2
Connections:
- net N$19 renamed P1.14
- net N$20 renamed P1.13
- net N$22 renamed P1.12
- net N$23 renamed P1.11
- net N$24 renamed P1.10
Changed lines of the file:
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@@
 <part name="C14" library="InkTime_v5" library_urn="urn:adsk.wipprod:fs.file:vf.MQzCYsgARiWfEyFJIY63Sg" deviceset="ESP32_C6_LIBRARY_1_ESP32_WROVER_EAGLE-LTSPICE_C" device="C0402" value="4.7uF"/>
 <part name="C15" library="InkTime_v5" library_urn="urn:adsk.wipprod:fs.file:vf.MQzCYsgARiWfEyFJIY63Sg" deviceset="ESP32_C6_LIBRARY_1_ESP32_WROVER_EAGLE-LTSPICE_C" device="C0402" value="1.0uF"/>
-<part name="U$6" library="InkTime_v5" library_urn="urn:adsk.wipprod:fs.file:vf.MQzCYsgARiWfEyFJIY63Sg" deviceset="NORDIC_NRF_1_XTAL_32KHZ" device="" value="32.768kHz"/>
+<part name="X2" library="InkTime_v5" library_urn="urn:adsk.wipprod:fs.file:vf.MQzCYsgARiWfEyFJIY63Sg" deviceset="NORDIC_NRF_1_XTAL_32KHZ" device="" value="32.768kHz"/>
 <part name="SUPPLY16" library="InkTime_v5" library_urn="urn:adsk.wipprod:fs.file:vf.MQzCYsgARiWfEyFJIY63Sg" deviceset="POWER_SYMBOLS_GND-BAR" device="" value="GND"/>
 <part name="SUPPLY17" library="InkTime_v5" library_urn="urn:adsk.wipprod:fs.file:vf.MQzCYsgARiWfEyFJIY63Sg" deviceset="POWER_SYMBOLS_GND-BAR" device="" value="GND"/>
@@
 <part name="C2" library="InkTime_v5" library_urn="urn:adsk.wipprod:fs.file:vf.MQzCYsgARiWfEyFJIY63Sg" deviceset="NORDIC_NRF_3_CAPACITOR" device="_0201_L" value="12pF"/>
 <part name="C1" library="InkTime_v5" library_urn="urn:adsk.wipprod:fs.file:vf.MQzCYsgARiWfEyFJIY63Sg" deviceset="NORDIC_NRF_3_CAPACITOR" device="_0201_L" value="12pF"/>
-<part name="U$13" library="InkTime_v5" library_urn="urn:adsk.wipprod:fs.file:vf.MQzCYsgARiWfEyFJIY63Sg" deviceset="NORDIC_NRF_XTAL_32MHZ" device=""/>
+<part name="X1" library="InkTime_v5" library_urn="urn:adsk.wipprod:fs.file:vf.MQzCYsgARiWfEyFJIY63Sg" deviceset="NORDIC_NRF_XTAL_32MHZ" device=""/>
 <part name="SUPPLY23" library="InkTime_v5" library_urn="urn:adsk.wipprod:fs.file:vf.MQzCYsgARiWfEyFJIY63Sg" deviceset="POWER_SYMBOLS_GND-BAR" device="" value="GND"/>
 <part name="SUPPLY24" library="InkTime_v5" library_urn="urn:adsk.wipprod:fs.file:vf.MQzCYsgARiWfEyFJIY63Sg" deviceset="POWER_SYMBOLS_GND-BAR" device="" value="GND"/>
@@
 <attribute name="VALUE" x="75.184" y="46.101" size="1.778" layer="96"/>
 </instance>
-<instance part="U$6" gate="X$1" x="-5.08" y="20.32" smashed="yes" rot="R270">
+<instance part="X2" gate="X$1" x="-5.08" y="20.32" smashed="yes" rot="R270">
 <attribute name="NAME" x="-8.89" y="20.32" size="1.778" layer="95" rot="R270"/>
 <attribute name="VALUE" x="-3.048" y="25.4" size="1.778" layer="96" rot="R270"/>
@@
 <attribute name="VALUE" x="195.199" y="-1.016" size="1.778" layer="96" rot="R90"/>
 </instance>
-<instance part="U$13" gate="X$1" x="182.88" y="2.54" smashed="yes" rot="R90">
+<instance part="X1" gate="X$1" x="182.88" y="2.54" smashed="yes" rot="R90">
 <attribute name="NAME" x="174.244" y="2.54" size="1.778" layer="95" rot="R90"/>
 <attribute name="VALUE" x="176.53" y="2.54" size="1.778" layer="96" rot="R90"/>
@@
 <junction x="200.66" y="-2.54"/>
 <pinref part="C1" gate="C$1" pin="2"/>
-<pinref part="U$13" gate="X$1" pin="2"/>
+<pinref part="X1" gate="X$1" pin="2"/>
 <wire x1="185.42" y1="5.08" x2="200.66" y2="5.08" width="0.1524" layer="91"/>
 <junction x="200.66" y="5.08"/>
-<pinref part="U$13" gate="X$1" pin="4"/>
+<pinref part="X1" gate="X$1" pin="4"/>
 <wire x1="185.42" y1="7.62" x2="200.66" y2="7.62" width="0.1524" layer="91"/>
 <junction x="200.66" y="7.62"/>
@@
 <wire x1="-10.16" y1="27.94" x2="-5.08" y2="27.94" width="0.1524" layer="91"/>
 <wire x1="-5.08" y1="27.94" x2="-5.08" y2="22.86" width="0.1524" layer="91"/>
-<pinref part="U$6" gate="X$1" pin="1"/>
+<pinref part="X2" gate="X$1" pin="1"/>
 <wire x1="-5.08" y1="27.94" x2="2.54" y2="27.94" width="0.1524" layer="91"/>
 <wire x1="2.54" y1="27.94" x2="2.54" y2="-7.62" width="0.1524" layer="91"/>
@@
 <net name="P0.01" class="0">
 <segment>
-<pinref part="U$6" gate="X$1" pin="2"/>
+<pinref part="X2" gate="X$1" pin="2"/>
 <wire x1="-5.08" y1="15.24" x2="-5.08" y2="10.16" width="0.1524" layer="91"/>
 <wire x1="-5.08" y1="10.16" x2="-10.16" y2="10.16" width="0.1524" layer="91"/>
@@
 </segment>
 </net>
-<net name="N$19" class="0">
+<net name="P1.14" class="0">
 <segment>
 <pinref part="U1" gate="G$1" pin="P1.14@B15"/>
 <wire x1="88.9" y1="12.7" x2="88.9" y2="17.78" width="0.1524" layer="91"/>
-</segment>
-</net>
-<net name="N$20" class="0">
+<label x="88.9" y="17.78" size="1.27" layer="95" rot="R90" xref="yes"/>
+</segment>
+</net>
+<net name="P1.13" class="0">
 <segment>
 <pinref part="U1" gate="G$1" pin="P1.13@A16"/>
 <wire x1="91.44" y1="12.7" x2="91.44" y2="17.78" width="0.1524" layer="91"/>
-</segment>
-</net>
-<net name="N$22" class="0">
+<label x="91.44" y="17.78" size="1.27" layer="95" rot="R90" xref="yes"/>
+</segment>
+</net>
+<net name="P1.12" class="0">
 <segment>
 <pinref part="U1" gate="G$1" pin="P1.12@B17"/>
 <wire x1="93.98" y1="12.7" x2="93.98" y2="17.78" width="0.1524" layer="91"/>
-</segment>
-</net>
-<net name="N$23" class="0">
+<label x="93.98" y="17.78" size="1.27" layer="95" rot="R90" xref="yes"/>
+</segment>
+</net>
+<net name="P1.11" class="0">
 <segment>
 <pinref part="U1" gate="G$1" pin="P1.11@B19"/>
 <wire x1="99.06" y1="12.7" x2="99.06" y2="17.78" width="0.1524" layer="91"/>
-</segment>
-</net>
-<net name="N$24" class="0">
+<label x="99.06" y="17.78" size="1.27" layer="95" rot="R90" xref="yes"/>
+</segment>
+</net>
+<net name="P1.10" class="0">
 <segment>
 <pinref part="U1" gate="G$1" pin="P1.10@A20"/>
 <wire x1="101.6" y1="12.7" x2="101.6" y2="17.78" width="0.1524" layer="91"/>
+<label x="101.6" y="17.78" size="1.27" layer="95" rot="R90" xref="yes"/>
 </segment>
 </net>
@@
 <net name="N$1" class="0">
 <segment>
-<pinref part="U$13" gate="X$1" pin="3"/>
+<pinref part="X1" gate="X$1" pin="3"/>
 <wire x1="180.34" y1="10.16" x2="180.34" y2="12.7" width="0.1524" layer="91"/>
 <wire x1="180.34" y1="12.7" x2="187.96" y2="12.7" width="0.1524" layer="91"/>
@@
 <net name="N$3" class="0">
 <segment>
-<pinref part="U$13" gate="X$1" pin="1"/>
+<pinref part="X1" gate="X$1" pin="1"/>
 <wire x1="180.34" y1="2.54" x2="180.34" y2="-2.54" width="0.1524" layer="91"/>
 <wire x1="180.34" y1="-2.54" x2="187.96" y2="-2.54" width="0.1524" layer="91"/>
